File: hardware/roller-shutter-controller.kicad_pcb (KiCad board)
At the start: 2 copper layers, 96 x 92 mm, 36 parts, among them J1 Screw_Terminal_01x06, J2 Screw_Terminal_01x04, J3 Screw_Terminal_01x10, K1 EC2-3NU, Q1 2N7000, Q2 2N7000, Q3 2N7000, U1 TSR_1-24120, U2 TSR_1-2433, U3 WeMos_C3_mini

Commit message: started work on new rev
Other:
- board text added: "CONTROLLER / POWER IN"
- board text added: "LOWER"
- board text added: "OUTSIDE / OUTPUTS"
- board text added: "VIN"
- board text added: "VIN Specification +12V with JP1 shorted +15-36V with JP1 open"
- board text removed: "+24V"
- board text removed: "CONTROLLER"
- board text removed: "OUTSIDE"

Commit message: first draft of v4 schematic
Other:
- board text added: "Roller Shutter RFID Access Dec 2025 Rev. C"
- board text removed: "Roller Shutter RFID Access Jan 2023 Rev. B"
Changed lines of the file:
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@@
 		)
 	)
-	(gr_text "Roller Shutter RFID Access\nJan 2023 Rev. B"
+	(gr_text "Roller Shutter RFID Access\nDec 2025 Rev. C"
 		(at 150.96 133.858 0)
 		(layer "F.SilkS" knockout)
