File: hardware/power.kicad_sch (KiCad schematic)
At the start: 23 parts, among them U5 LMR50410, U6 LMR50410

Commit message: wip
Parts:
- C10, C11, C5, C6, C9: DigiKey (none) -> 445-5968-1-ND
- C7, C8: DigiKey (none) -> 490-10672-1-ND; MPN (none) -> GCM155R71H104KE02D; Manufacturer (none) -> Murata
- D4: DigiKey (none) -> 732-4971-1-ND; MPN (none) -> 150060GS75000; Manufacturer (none) -> Wurth
- F1: DigiKey (none) -> SF-0603S040-2CT-ND
- L1: DigiKey (none) -> SRR1210-330MCT-ND
- L2: DigiKey (none) -> SRP5030T-100MCT-ND
- R10: DigiKey (none) -> 541-4089-1-ND; MPN (none) -> CRCW040269K8FKEDC; Manufacturer (none) -> Vishay
- R11, R9: DigiKey (none) -> 541-4088-1-ND; MPN (none) -> CRCW040222K1FKEDC; Manufacturer (none) -> Vishay
- R12: DigiKey (none) -> 541-4064-1-ND; MPN (none) -> CRCW0402220RFKEDC; Manufacturer (none) -> Vishay
- R8: Digikey (none) -> 541-309KLCT-ND; MPN (none) -> CRCW0402309KFKED; Manufacturer (none) -> Vishay
- U5, U6: DigiKey (none) -> 296-LMR50410XFDBVRCT-ND; MPN (none) -> LMR50410XFDBVR; Manufacturer (none) -> TI
Other:
- note removed: "TODO: add MPN, SPN, Manufacturer to all parts"
